File: Hardware/PFC-LLC Board/KiCAD Simulations.sch (KiCad schematic (older format))
At the start: 44 parts, among them J1 1792229, J2 Conn_01x02_Female, J3 1792229, Q1 C2M0160120D, U1 UCC28180DR

Commit message: PFC Gerber files generated
Parts:
- J2: footprint Connector_PinHeader_1.27mm:PinHeader_1x02_P1.27mm_Vertical -> Connector_PinHeader_2.54mm:PinHeader_1x02_P2.54mm_Vertical
Changed lines of the file:
@@
 F 0 "J2" H 642 3775 50  0000 C CNN
 F 1 "Conn_01x02_Female" H 642 3866 50  0000 C CNN
-F 2 "Connector_PinHeader_1.27mm:PinHeader_1x02_P1.27mm_Vertical" H 750 4100 50  0001 C CNN
+F 2 "Connector_PinHeader_2.54mm:PinHeader_1x02_P2.54mm_Vertical" H 750 4100 50  0001 C CNN
 F 3 "~" H 750 4100 50  0001 C CNN
 	1    750  4100
