File: Hardware/PFC-LLC Board/KiCAD Simulations.kicad_pcb (KiCad board)
At the start: 2 copper layers, 127 parts, among them J1 1792229, J2 Conn_01x02_Female, J3 PFC OUT, J4 LLC IN, J5 Conn_01x02_Female, J6 1792229, Q1 C2M0160120D, U1 UCC28180DR, U1LLC1 UCC256403DDBR, U2LLC1 UCC24624DT

Commit message: PFC Gerber files generated
Parts:
- removed C16: 220p, Capacitor_SMD:C_0402_1005Metric_Pad0.74x0.62mm_HandSolder
- removed Cboot1: 220n, Capacitor_SMD:C_0603_1608Metric_Pad1.08x0.95mm_HandSolder
- removed Cbw1: 3.9p, Capacitor_SMD:C_0402_1005Metric_Pad0.74x0.62mm_HandSolder
- removed Ccomp3: 390n, Capacitor_SMD:C_1206_3216Metric_Pad1.33x1.80mm_HandSolder
- removed Cin2: 47u, Capacitor_THT:CP_Radial_D25.0mm_P10.00mm_SnapIn
- removed Cinx1: 1.5u, Capacitor_THT:C_Rect_L26.5mm_W10.5mm_P22.50mm_MKS4
- removed Cisns1: 3.3p, Capacitor_SMD:C_0402_1005Metric_Pad0.74x0.62mm_HandSolder
- removed Cisns2: 150p, LLC_Cisns2:FA26C0G2J151JNU00
- removed Cout21, Cout22, Cout23, Cout24, Cout25, Cout26: 120u, LLC_Cout:35SVPF120M
- removed Coutx21, Coutx22, Coutx23, Coutx24: 22u, Capacitor_SMD:C_0805_2012Metric_Pad1.18x1.45mm_HandSolder
- removed Cr1, Cr2: 33.454n, Capacitor_THT:C_Rect_L13.0mm_W5.0mm_P10.00mm_FKS3_FKP3_MKS4
- removed Creg1: 2.2u, Capacitor_SMD:C_0402_1005Metric_Pad0.74x0.62mm_HandSolder
- removed Crvcc2, Cvrcc1: 4.7u, Capacitor_SMD:C_0805_2012Metric_Pad1.18x1.45mm_HandSolder
- removed Css11, Css12, Css13: 47n, Capacitor_SMD:C_0402_1005Metric_Pad0.74x0.62mm_HandSolder
- removed Cvcc21, Cvcc22, Cvcc23, Cvcc24, Cvcc25, Cvcc26, Cvcc27, Cvcc28: 15u, Capacitor_SMD:CP_Elec_5x5.8
- removed Cvcc3: 2.2u, Capacitor_SMD:C_0805_2012Metric_Pad1.18x1.45mm_HandSolder
- removed Cvcr1: 66.044p, Capacitor_THT:C_Rect_L7.2mm_W4.5mm_P5.00mm_FKS2_FKP2_MKS2_MKP2
- removed Cvcr21, Cvcr22, Cvcr23, Cvcr24, Cvcr25, Cvcr26: 1n, Capacitor_SMD:C_0805_2012Metric_Pad1.18x1.45mm_HandSolder
- removed Cz1: 100n, Capacitor_SMD:C_0603_1608Metric_Pad1.08x0.95mm_HandSolder
- removed Dboot1: DIODE, DO-214BA:DO-214BA
- removed Dz1: BZX84Cxx, Diode_SMD:D_SOT-23_ANK
- removed J4: LLC IN, Connector2x1:PHOENIX_1792229
- removed J5: Conn_01x02_Female, Connector_PinHeader_1.27mm:PinHeader_1x02_P1.27mm_Vertical
- removed J6: 1792229, Connector2x1:PHOENIX_1792229
- removed Lr1: PA4344.473ANLT, LLC_Lr:PA4344.473ANLT
- removed QM1, QM2: IPP060N06N, Package_TO_SOT_THT:TO-220-3_Vertical
- removed QM3, QM4: C2M0025120D, Package_TO_SOT_THT:TO-247-3_Vertical
- removed R19: 121k, Resistor_SMD:R_0402_1005Metric_Pad0.72x0.64mm_HandSolder
- removed R20, R27, R28: 4.99M, Resistor_SMD:R_1206_3216Metric_Pad1.30x1.75mm_HandSolder
- removed Rbias1: 6.04k, Resistor_SMD:R_0402_1005Metric_Pad0.72x0.64mm_HandSolder
- removed Rboot1: 2.20, Resistor_SMD:R_0805_2012Metric_Pad1.20x1.40mm_HandSolder
- removed Rbw1: 35.7k, Resistor_SMD:R_0402_1005Metric_Pad0.72x0.64mm_HandSolder
- removed Rbw2: 10k, Resistor_SMD:R_0201_0603Metric_Pad0.64x0.40mm_HandSolder
- removed Rcomp2, Rvcc1: 44.2k, Resistor_SMD:R_0201_0603Metric_Pad0.64x0.40mm_HandSolder
- removed Rdrv1, Rdrv2: 5.11k, Resistor_SMD:R_0402_1005Metric_Pad0.72x0.64mm_HandSolder
- removed Rfbb2: 8.06k, Resistor_SMD:R_0402_1005Metric_Pad0.72x0.64mm_HandSolder
- removed Rfbt4: 110k, Resistor_SMD:R_0603_1608Metric_Pad0.98x0.95mm_HandSolder
- removed Rho1, Rlo1: 1, Resistor_SMD:R_0402_1005Metric_Pad0.72x0.64mm_HandSolder
- removed Risns1: 80.759, Resistor_SMD:R_0603_1608Metric_Pad0.98x0.95mm_HandSolder
- removed Rled1: 36.5k, Resistor_SMD:R_0201_0603Metric_Pad0.64x0.40mm_HandSolder
- removed Rlimit1: 18.2k, Resistor_SMD:R_1206_3216Metric_Pad1.30x1.75mm_HandSolder
- removed Rvcc2: 12.1k, Resistor_SMD:R_0201_0603Metric_Pad0.64x0.40mm_HandSolder
- removed TPblk1, TPho1, TPhs1, TPisns1, TPlo1: TestPoint, TestPoint:TestPoint_Pad_D1.0mm
- removed TPgnd3, TPgnd4: TestPoint GND, TestPoint:TestPoint_Pad_D1.0mm
- removed TR1: TRANSF6, LLC_T1:EPCOS-B65982E0012D001-MFG
- removed U1LLC1: UCC256403DDBR, LLC_U1:UCC256403DDBR
- removed U2LLC1: UCC24624DT, LLC_U2:UCC24624DT
- removed UO1: PS2501L-1-F3-A, LLC_O1:PS2501L-1-F3-A
- removed UVR1: TLV431AIDBVT, LLC_VR1:TLV431AIDBVT
- J2: footprint Connector_PinHeader_1.27mm:PinHeader_1x02_P1.27mm_Vertical -> Connector_PinHeader_2.54mm:PinHeader_1x02_P2.54mm_Vertical
- J3: value PFC OUT -> 1792229
- TPQ1: value TP Q1 -> TestPoint Q1
- TPgnd5: value TP GND Q1 -> TestPoint GND Q1
- moved TPgnd1 64.3 mm to (146.1, 82.3)
- moved Dturnoff1 42.0 mm to (165.6, 56.4)
- moved Rgate1 42.0 mm to (156.7, 63.4)
- moved Rgate2 42.0 mm to (166.2, 63.4)
- moved Rgate3 42.0 mm to (156.7, 56.4)
- moved J2 40.0 mm to (191.0, 78.7)
- moved Rfbt3 38.1 mm to (193.7, 57.4)
- moved Cisense1 38.1 mm to (140.3, 71.4)
- moved Coutx2 38.1 mm to (193.7, 40.9)
- moved Dboost1 38.1 mm to (120.7, 72.0)
- moved Dstart1 38.1 mm to (120.7, 81.5)
- moved Rfbt1 38.1 mm to (193.7, 66.3)
- moved TPDstart1 38.1 mm to (109.9, 88.5)
- moved TPDstart2 38.1 mm to (120.7, 90.4)
- moved TPisense1 38.1 mm to (140.3, 65.0)
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Routing:
- net GND: track 795.5 -> 371.8 mm, vias 4 -> 3
- net Net-(Cout21-Pad1): track 305.9 -> 0.00 mm, vias 3 -> 0
- net GND1: track 242.3 -> 0.00 mm, vias 23 -> 0
- net Net-(Cvcc21-Pad1): track 176.0 -> 0.00 mm, vias 2 -> 0
- net /LLC/HS: track 162.0 -> 0.00 mm, vias 1 -> 0
- net Net-(Cisns2-Pad2): track 160.7 -> 0.00 mm, vias 2 -> 0
- net Net-(Cin2-Pad1): track 140.6 -> 0.00 mm, vias 1 -> 0
- net Net-(QM3-Pad3): track 139.2 -> 0.00 mm, vias 16 -> 0
- net Net-(Lr1-Pad1): track 106.7 -> 0.00 mm, vias 5 -> 0
- net Net-(QM4-Pad2): track 103.8 -> 0.00 mm
- net /LLC/LO: track 93.1 -> 0.00 mm, vias 3 -> 0
- net Net-(Cvcr1-Pad2): track 84.1 -> 0.00 mm
- net /LLC/HO: track 79.2 -> 0.00 mm, vias 2 -> 0
- net Net-(Cisns1-Pad1): track 65.2 -> 0.00 mm, vias 2 -> 0
- net Net-(Rbw1-Pad1): track 49.9 -> 0.00 mm, vias 1 -> 0
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- removed copper zone on B.Cu, net GND1
- removed copper zone on F.Cu, net GND1
- removed copper zone on B.Cu, net Net-(Cout21-Pad1)
- removed copper zone on F.Cu, net Net-(Cout21-Pad1)
- removed copper zone on B.Cu, net Net-(Lr1-Pad1)
- removed copper zone on F.Cu, net Net-(Lr1-Pad1)
- removed copper zone on B.Cu, net Net-(QM3-Pad3)
- removed copper zone on F.Cu, net Net-(QM3-Pad3)
- removed copper zone on B.Cu, net Net-(QM4-Pad2)
Other:
- board outline added: 210.8 x 69.6 mm

Commit message: Gerber files regenerated
Parts:
- moved TPDstart1 79.0 mm to (158.8, 26.4)
- moved TPDstart2 68.6 mm to (145.3, 26.4)
- moved J1 60.1 mm to (106.4, 83.1), turned to 270 degrees
- moved Rntc1 56.7 mm to (95.0, 83.1), turned to 270 degrees
- moved L1 50.2 mm to (126.7, 50.7), turned to 90 degrees
- moved Dboost1 48.1 mm to (135.9, 26.4)
- moved Dstart1 47.7 mm to (142.0, 38.9), turned to 0 degrees
- moved Uac1 44.0 mm to (98.2, 73.5), turned to 0 degrees
- moved Cin1 37.7 mm to (105.8, 65.9), turned to 90 degrees
Routing:
- net Net-(Dboost1-Pad2): track 116.4 -> 77.8 mm, vias 1 -> 0
- net Net-(Coutx1-Pad1): track 161.9 -> 131.4 mm
- net Net-(Cin1-Pad1): track 77.9 -> 83.2 mm, vias 1 -> 0
- net Net-(Cin1-Pad2): track 147.3 -> 142.4 mm
Other:
- board size 210.8 x 69.6 mm -> 157 x 79.5 mm
