File: Hardware/PFC-LLC Board/LLC.sch (KiCad schematic (older format))
At the start: 83 parts, among them J4 1792229, J5 Conn_01x02_Female, J6 1792229, U1LLC1 UCC256403DDBR, U2LLC1 UCC24624DT

Commit message: LLC footprints and schematic update
No transformer yet
Parts:
- removed Cisns2: 150p, LLC_Cisns2:FA26C0G2J151JNU00, symbol KiCAD-Simulations-rescue:FA26C0G2J151JNU00-LLC_Cisns2
- removed Creg1: 2.2u, Capacitor_SMD:C_0402_1005Metric_Pad0.74x0.62mm_HandSolder, symbol KiCAD-Simulations-rescue:C-Device
- removed Css12, Css13: 47n, Capacitor_SMD:C_0402_1005Metric_Pad0.74x0.62mm_HandSolder, symbol KiCAD-Simulations-rescue:C-Device
- removed Cvcc21, Cvcc22, Cvcc23, Cvcc24, Cvcc25, Cvcc26, Cvcc27, Cvcc28: 15u, Capacitor_SMD:CP_Elec_5x5.8, symbol KiCAD-Simulations-rescue:CP-Device
- removed Cvcr22, Cvcr23, Cvcr24, Cvcr25, Cvcr26: 1n, Capacitor_SMD:C_0805_2012Metric_Pad1.18x1.45mm_HandSolder, symbol KiCAD-Simulations-rescue:C-Device
- removed Lr1: PA4344.473ANLT, LLC_Lr:PA4344.473ANLT, symbol KiCAD-Simulations-rescue:PA4344.473ANLT-LLC_Lr
- removed QM3, QM4: C2M0025120D, Package_TO_SOT_THT:TO-247-3_Vertical, symbol KiCAD-Simulations-rescue:C2M0025120D-Transistor_FET
- removed U2LLC1: UCC24624DT, LLC_U2:UCC24624DT, symbol KiCAD-Simulations-rescue:UCC24624DT-LLC_U2
- added CbootB: 470n, Capacitor_SMD:C_0603_1608Metric_Pad1.08x0.95mm_HandSolder, symbol KiCAD-Simulations-rescue:C-Device
- added CbwB: 12p, Capacitor_SMD:C_1206_3216Metric_Pad1.33x1.80mm_HandSolder, symbol KiCAD-Simulations-rescue:C-Device
- added Cisns2: 220p, Capacitor_SMD:C_1206_3216Metric_Pad1.33x1.80mm_HandSolder, symbol Device:C
- added Cpfc: 450HXW100MEFR16X30, LLC_pfc:450HXW100MEFR16X30, symbol LLC_pfc:450HXW100MEFR16X30
- added Cvcc2A, Cvcc2B, Cvcc2C, Cvcc2D, Cvcc2E, Cvcc2F, Cvcc2G, Cvcc2H: UUD1V150MCL1GS, LLC_Cvcc2:UUD1V150MCL1GS, symbol LLC_Cvcc2:UUD1V150MCL1GS
- added Dsec, Dsec2: D_Schottky, LLC_Dsec:STPS30M60DJF-TR, symbol Device:D_Schottky
- added Lr: 2100LL-180-H-RC, LLC_Lr:2100LL-180-H-RC, symbol LLC_Lr:2100LL-180-H-RC
- added Rbw1B: 82k, Resistor_SMD:R_2512_6332Metric_Pad1.40x3.35mm_HandSolder, symbol KiCAD-Simulations-rescue:R-Device
- C16: footprint Capacitor_SMD:C_0402_1005Metric_Pad0.74x0.62mm_HandSolder -> Capacitor_SMD:C_1206_3216Metric_Pad1.33x1.80mm_HandSolder
- CbootA: renamed from Cboot1; value 220n -> 470n
- CbwA: renamed from Cbw1; value 3.9p -> 12p; footprint Capacitor_SMD:C_0402_1005Metric_Pad0.74x0.62mm_HandSolder -> Capacitor_SMD:C_1206_3216Metric_Pad1.33x1.80mm_HandSolder
- Ccomp: renamed from Ccomp3; value 390n -> 2.7n
- Cin: renamed from Cin2; footprint Capacitor_THT:CP_Radial_D25.0mm_P10.00mm_SnapIn -> Capacitor_THT:CP_Radial_D22.0mm_P10.00mm_SnapIn
- Cisns: renamed from Cisns1; footprint Capacitor_SMD:C_0402_1005Metric_Pad0.74x0.62mm_HandSolder -> Capacitor_SMD:C_0805_2012Metric_Pad1.18x1.45mm_HandSolder
- CoutxA: renamed from Coutx21; footprint Capacitor_SMD:C_0805_2012Metric_Pad1.18x1.45mm_HandSolder -> Capacitor_SMD:C_1206_3216Metric_Pad1.33x1.80mm_HandSolder
- CoutxB: renamed from Coutx22; footprint Capacitor_SMD:C_0805_2012Metric_Pad1.18x1.45mm_HandSolder -> Capacitor_SMD:C_1206_3216Metric_Pad1.33x1.80mm_HandSolder
- CoutxC: renamed from Coutx23; footprint Capacitor_SMD:C_0805_2012Metric_Pad1.18x1.45mm_HandSolder -> Capacitor_SMD:C_1206_3216Metric_Pad1.33x1.80mm_HandSolder
- CoutxD: renamed from Coutx24; footprint Capacitor_SMD:C_0805_2012Metric_Pad1.18x1.45mm_HandSolder -> Capacitor_SMD:C_1206_3216Metric_Pad1.33x1.80mm_HandSolder
- Cr1, Cr2: value 33.454n -> 150n; footprint Capacitor_THT:C_Rect_L13.0mm_W5.0mm_P10.00mm_FKS3_FKP3_MKS4 -> Capacitor_SMD:C_2220_5650Metric_Pad1.97x5.40mm_HandSolder
- Css: renamed from Css11; value 47n -> 150n; footprint Capacitor_SMD:C_0402_1005Metric_Pad0.74x0.62mm_HandSolder -> Capacitor_SMD:C_1206_3216Metric_Pad1.33x1.80mm_HandSolder
- Cvcc: renamed from Cvcc3; footprint Capacitor_SMD:C_0603_1608Metric_Pad1.08x0.95mm_HandSolder -> Capacitor_SMD:C_1206_3216Metric_Pad1.33x1.80mm_HandSolder
- Cvcr1: value 66.044p -> 220p; footprint Capacitor_THT:C_Rect_L7.2mm_W4.5mm_P5.00mm_FKS2_FKP2_MKS2_MKP2 -> Capacitor_SMD:C_1206_3216Metric_Pad1.33x1.80mm_HandSolder
- Cvcr2: renamed from Cvcr21; value 1n -> 22n; footprint Capacitor_SMD:C_0805_2012Metric_Pad1.18x1.45mm_HandSolder -> Capacitor_SMD:C_1206_3216Metric_Pad1.33x1.80mm_HandSolder
- Cz: renamed from Cz1; footprint Capacitor_SMD:C_0603_1608Metric_Pad1.08x0.95mm_HandSolder -> Capacitor_SMD:C_1206_3216Metric_Pad1.33x1.80mm_HandSolder
- Dboot: renamed from Dboot1; footprint DO-214BA:DO-214BA -> Diode_THT:D_DO-34_SOD68_P7.62mm_Horizontal
- J5: footprint Connector_PinHeader_1.27mm:PinHeader_1x02_P1.27mm_Vertical -> Connector_PinHeader_2.54mm:PinHeader_1x02_P2.54mm_Vertical
- R19: value 121k -> 2.7k; footprint Resistor_SMD:R_0402_1005Metric_Pad0.72x0.64mm_HandSolder -> Resistor_SMD:R_2512_6332Metric_Pad1.40x3.35mm_HandSolder
- R20, R27: value 4.99M -> 120k; footprint Resistor_SMD:R_1206_3216Metric_Pad1.30x1.75mm_HandSolder -> Resistor_SMD:R_2512_6332Metric_Pad1.40x3.35mm_HandSolder
- R28: value 4.99M -> 100k; footprint Resistor_SMD:R_1206_3216Metric_Pad1.30x1.75mm_HandSolder -> Resistor_SMD:R_2512_6332Metric_Pad1.40x3.35mm_HandSolder
- Rbias: renamed from Rbias1; footprint Resistor_SMD:R_0402_1005Metric_Pad0.72x0.64mm_HandSolder -> Resistor_SMD:R_2512_6332Metric_Pad1.40x3.35mm_HandSolder
- Rboot: renamed from Rboot1; footprint Resistor_SMD:R_0805_2012Metric_Pad1.20x1.40mm_HandSolder -> Resistor_SMD:R_2512_6332Metric_Pad1.40x3.35mm_HandSolder
- Rbw1A: renamed from Rbw1; value 35.7k -> 82k; footprint Resistor_SMD:R_0402_1005Metric_Pad0.72x0.64mm_HandSolder -> Resistor_SMD:R_2512_6332Metric_Pad1.40x3.35mm_HandSolder
- Rbw2: footprint Resistor_SMD:R_0201_0603Metric_Pad0.64x0.40mm_HandSolder -> Resistor_SMD:R_2512_6332Metric_Pad1.40x3.35mm_HandSolder
- Rcomp: renamed from Rcomp2; value 44.2k -> 18.7k; footprint Resistor_SMD:R_0201_0603Metric_Pad0.64x0.40mm_HandSolder -> Resistor_SMD:R_2512_6332Metric_Pad1.40x3.35mm_HandSolder
- Rdrv1, Rdrv2: footprint Resistor_SMD:R_0402_1005Metric_Pad0.72x0.64mm_HandSolder -> Resistor_SMD:R_2512_6332Metric_Pad1.40x3.35mm_HandSolder
- Rfbb: renamed from Rfbb2; footprint Resistor_SMD:R_0402_1005Metric_Pad0.72x0.64mm_HandSolder -> Resistor_SMD:R_2512_6332Metric_Pad1.40x3.35mm_HandSolder
- Rfbt: renamed from Rfbt4; footprint Resistor_SMD:R_0603_1608Metric_Pad0.98x0.95mm_HandSolder -> Resistor_SMD:R_2512_6332Metric_Pad1.40x3.35mm_HandSolder
- Rho: renamed from Rho1; footprint Resistor_SMD:R_0402_1005Metric_Pad0.72x0.64mm_HandSolder -> Resistor_SMD:R_2512_6332Metric_Pad1.40x3.35mm_HandSolder
- Risns: renamed from Risns1; value 80.759 -> 390; footprint Resistor_SMD:R_0603_1608Metric_Pad0.98x0.95mm_HandSolder -> Resistor_SMD:R_2512_6332Metric_Pad1.40x3.35mm_HandSolder
- Rled: renamed from Rled1; footprint Resistor_SMD:R_0201_0603Metric_Pad0.64x0.40mm_HandSolder -> Resistor_SMD:R_2512_6332Metric_Pad1.40x3.35mm_HandSolder
- Rlimit: renamed from Rlimit1; footprint Resistor_SMD:R_1206_3216Metric_Pad1.30x1.75mm_HandSolder -> Resistor_SMD:R_2512_6332Metric_Pad1.40x3.35mm_HandSolder
- Rlo: renamed from Rlo1; footprint Resistor_SMD:R_0402_1005Metric_Pad0.72x0.64mm_HandSolder -> Resistor_SMD:R_2512_6332Metric_Pad1.40x3.35mm_HandSolder
- Rvcc1: value 44.2k -> 220k; footprint Resistor_SMD:R_0201_0603Metric_Pad0.64x0.40mm_HandSolder -> Resistor_SMD:R_2512_6332Metric_Pad1.40x3.35mm_HandSolder
- Rvcc2: value 12.1k -> 1.2M; footprint Resistor_SMD:R_0201_0603Metric_Pad0.64x0.40mm_HandSolder -> Resistor_SMD:R_2512_6332Metric_Pad1.40x3.35mm_HandSolder
- renumbered Cinx1 to Cinx, Cout21 to CoutA, Cout22 to CoutB, Cout23 to CoutC, Cout24 to CoutD, Cout25 to CoutE, Cout26 to CoutF, Dz1 to Dz, UVR1 to UVR
Connections:
- net GND: now also CbwB.2, Cpfc.2, Cvcc2A.2, Cvcc2B.2, Cvcc2C.2, Cvcc2D.2, Cvcc2E.2, Cvcc2F.2, Cvcc2G.2, Cvcc2H.2; no longer CbwA.2
- net GND1: now also TR1.6, TR1.7
- net HS: now also CbootB.1, Lr.2
- net at Cin.1, Cinx.1, Cr1.1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: now also Cpfc.1
- net at Cr1.2, Cr2.1, Cvcr1.1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: now also Cisns2.1
- net at Cisns.1, Risns.1, TPisns1.1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: now also Cisns2.2
- net at CbwA.1, Rbw1A.2, Rbw2.1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: now also Rbw1B.2
- net at Rbw1A.1, TR1.3: now also Rbw1B.1
- net at CbootA.2, Dboot.2 (A), U1LLC1.14 (HB): now also CbootB.2
- net at Cvcc.1, J5.2 (Pin_2), U1LLC1.3 (VCC): now also Cvcc2A.1, Cvcc2B.1, Cvcc2C.1, Cvcc2D.1, Cvcc2E.1, Cvcc2F.1, Cvcc2G.1, Cvcc2H.1
- net at CoutA.1, CoutB.1, CoutC.1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: now also Dsec.1 (K), Dsec2.1 (K); no longer TR1.6, TR1.7
- net at TR1.1: now also Lr.1
- net at TR1.5: now also Dsec2.2 (A)
- net at TR1.8: now also Dsec.2 (A)
- new net: CbwA.2, CbwB.1
Other:
- moved on the sheet: C16, CbootA, CbwA, Ccomp, Cin, Cinx, Cisns, CoutA, CoutB, CoutC, CoutD, CoutE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
