File: Hardware/PFC-LLC Board/LLC.sch (KiCad schematic (older format))
At the start: 78 parts, among them J4 1792229, J5 Conn_01x02_Female, J6 1792229, U1LLC1 UCC256403DDBR

Commit message: LLC PCB ready w/ PFC board
Parts:
- removed Cinx: 1.5u, Capacitor_THT:C_Rect_L26.5mm_W10.5mm_P22.50mm_MKS4, symbol KiCAD-Simulations-rescue:C-Device
- removed Dsec, Dsec2: D_Schottky, LLC_Dsec:STPS30M60DJF-TR, symbol Device:D_Schottky
- removed TR1: TRANSF6, LLC_T1:EPCOS-B65982E0012D001-MFG, symbol KiCAD-Simulations-rescue:TRANSF6-Transformer
- added Dsec1, Dsec2: STPS30M60DJF-TR, LLC_Dsec:STPS30M60DJF-TR-Modified, symbol LLC_Dsec:STPS30M60DJF-TR
- added TPgnd6, TPisoGND1: TestPoint, Connector_PinHeader_2.54mm:PinHeader_1x01_P2.54mm_Vertical, symbol Connector:TestPoint
- added TPllc1, TPpfc1: TestPoint, TestPoint:TestPoint_THTPad_D4.0mm_Drill2.0mm, symbol Connector:TestPoint
- added TR1: TRANSF6-WE, LLC_Transformer:Transformer, symbol LLC_Transformer:TRANSF6-WE
- renumbered CbootA to CbootA1, CbootB to CbootB1, CbwA to CbwA1, CbwB to CbwB1, Ccomp to Ccomp3, Cin to Cin2, Cisns to Cisns1, CoutA to CoutA1, CoutB to CoutB1, CoutC to CoutC1, CoutD to CoutD1, CoutE to CoutE1, CoutF to CoutF1, CoutxA to CoutxA1, CoutxB to CoutxB1, CoutxC to CoutxC1, CoutxD to CoutxD1, Cpfc to Cpfc1, Css to Css1, Cvcc to Cvcc2, Cvcc2A to Cvcc2A1, Cvcc2B to Cvcc2B1, Cvcc2C to Cvcc2C1, Cvcc2D to Cvcc2D1, Cvcc2E to Cvcc2E1, Cvcc2F to Cvcc2F1, Cvcc2G to Cvcc2G1, Cvcc2H to Cvcc2H1, Cz to Cz1, Dboot to Dboot1, Dz to Dz1, Lr to Lr1, UO1 to O1, Rbias to Rbias1, Rboot to Rboot1, Rbw1A to Rbw1A1, Rbw1B to Rbw1B1, Rcomp to Rcomp2, Rfbb to Rfbb2, Rfbt to Rfbt4, Rho to Rho1, Risns to Risns1, Rled to Rled1, Rlimit to Rlimit1, Rlo to Rlo1, UVR to VR1
Connections:
- net GND: now also TPgnd6.1, TR1.6
- net GND1: now also TPisoGND1.1, TR1.11, TR1.12, TR1.13, TR1.14
- net at Cin2.1, Cr1.1, QM1.2 (D)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: now also TPllc1.1; no longer Cpfc1.1, J4.2
- net at Cisns2.1, Cr1.2, Cr2.1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: now also TR1.2
- net at Rbw1A1.1, Rbw1B1.1: now also TR1.7
- net at CoutA1.1, CoutB1.1, CoutC1.1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: now also Dsec1.5, Dsec1.6, Dsec1.7, Dsec1.8, Dsec2.5, Dsec2.6, Dsec2.7, Dsec2.8
- net at Lr1.1: now also TR1.4
- new net: Cpfc1.1, J4.2, TPpfc1.1
- new net: Dsec1.1, Dsec1.2, Dsec1.3, Dsec1.4, TR1.10, TR1.9
- new net: Dsec2.1, Dsec2.2, Dsec2.3, Dsec2.4, TR1.15, TR1.16
Other:
- moved on the sheet: Cin2, CoutA1, CoutB1, CoutC1, CoutD1, CoutE1, CoutF1, CoutxA1, CoutxB1, CoutxC1, CoutxD1, Cpfc1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

Commit message: LLC gerber files regenerated
2512 footprints updated to 1206 for Rlimit, Rcomp, drv1, drv2
Parts:
- Rcomp2, Rdrv1, Rdrv2, Rlimit1: footprint Resistor_SMD:R_2512_6332Metric_Pad1.40x3.35mm_HandSolder -> Resistor_SMD:R_1206_3216Metric_Pad1.30x1.75mm_HandSolder
Changed lines of the file:
@@
 F 0 "Rdrv1" H 4420 1846 50  0000 L CNN
 F 1 "5.11k" H 4420 1755 50  0000 L CNN
-F 2 "Resistor_SMD:R_2512_6332Metric_Pad1.40x3.35mm_HandSolder" V 4280 1800 50  0001 C CNN
+F 2 "Resistor_SMD:R_1206_3216Metric_Pad1.30x1.75mm_HandSolder" V 4280 1800 50  0001 C CNN
 F 3 "~" H 4350 1800 50  0001 C CNN
 	1    4350 1800
@@
 F 0 "Rdrv2" H 4420 2846 50  0000 L CNN
 F 1 "5.11k" H 4420 2755 50  0000 L CNN
-F 2 "Resistor_SMD:R_2512_6332Metric_Pad1.40x3.35mm_HandSolder" V 4280 2800 50  0001 C CNN
+F 2 "Resistor_SMD:R_1206_3216Metric_Pad1.30x1.75mm_HandSolder" V 4280 2800 50  0001 C CNN
 F 3 "~" H 4350 2800 50  0001 C CNN
 	1    4350 2800
@@
 F 0 "Rcomp2" V 14343 6500 50  0000 C CNN
 F 1 "18.7k" V 14434 6500 50  0000 C CNN
-F 2 "Resistor_SMD:R_2512_6332Metric_Pad1.40x3.35mm_HandSolder" V 14480 6500 50  0001 C CNN
+F 2 "Resistor_SMD:R_1206_3216Metric_Pad1.30x1.75mm_HandSolder" V 14480 6500 50  0001 C CNN
 F 3 "~" H 14550 6500 50  0001 C CNN
 	1    14550 6500
@@
 F 0 "Rlimit1" V 15193 5000 50  0000 C CNN
 F 1 "18.2k" V 15284 5000 50  0000 C CNN
-F 2 "Resistor_SMD:R_2512_6332Metric_Pad1.40x3.35mm_HandSolder" V 15330 5000 50  0001 C CNN
+F 2 "Resistor_SMD:R_1206_3216Metric_Pad1.30x1.75mm_HandSolder" V 15330 5000 50  0001 C CNN
 F 3 "~" H 15400 5000 50  0001 C CNN
 	1    15400 5000
